File: hw/pcb/mark3/mark3.kicad_pcb (KiCad board)
At the start: 2 copper layers, 100.1 x 65 mm, 68 parts, among them P1 CONN_02X05, P2 USB_A, P3 CONN_02X05, P4 CONN_02X20, P5 USB_A, Q1 MMBT3904, Q2 MMBT3904, SW1 SW_Push, SW2 SW_Push, U1 AMS1117-2.5, U2 AMS1117-3.3, U3 AMS1117-1.2, U4 EP4CE10E22C8N, U6 HY57V561620, U7 W25Q32FVSSIQ, Y1 Crystal_GND23

Commit message: WIP
Parts:
- removed C1, C2, C3: 10uF, SMD_Packages:SMD-1206_Pol
- removed C10, C11, C12, C13, C14, C15, C16, C17, C18, C19, C20, C21, C22, C23, C24, C25, C26, C27, C28, C29, C30, C34, C35, C36, C37, C38, C39, C40, C41, C7, C8, C9: 100nF, Capacitors_SMD:C_0805_HandSoldering
- removed C4, C5, C6: 100uF, Capacitors_SMD:c_elec_6.3x7.7
- removed D1, D2, D3: LED, LEDs:LED_0805
- removed P1, P3: CONN_02X05, Connectors:IDC_Header_Straight_10pins
- removed P2, P5: USB_A, Connectors:USB_A
- removed P4: CONN_02X20, Connectors:IDC_Header_Straight_40pins
- removed Q1, Q2: MMBT3904, SOT-23
- removed R1, R16, R2, R20: 1K, Resistors_SMD:R_0805_HandSoldering
- removed R10, R11, R12, R14, R15: 10K, Resistors_SMD:R_0805_HandSoldering
- removed R13: 33, Resistors_SMD:R_0805_HandSoldering
- removed R21: 1k, Resistors_SMD:R_0805_HandSoldering
- removed SW1, SW2: SW_Push, Buttons_Switches_ThroughHole:SW_PUSH_6mm_h4.3mm
- removed U1: AMS1117-2.5, TO_SOT_Packages_SMD:SOT-223
- removed U2: AMS1117-3.3, TO_SOT_Packages_SMD:SOT-223
- removed U3: AMS1117-1.2, TO_SOT_Packages_SMD:SOT-223
- removed U7: W25Q32FVSSIQ, SMD_Packages:SOIC-8-N
- removed Y1: Crystal_GND23, footprints:Crystal_SMD_7050_4Pads_R
- moved U6 152.9 mm to (228.3, 75.4)
- moved U4 147.9 mm to (229.0, 51.1)
Routing:
- net VCC3p3: track 531.9 -> 0.00 mm, vias 38 -> 0
- net VCC2p5: track 140.5 -> 1.37 mm, vias 4 -> 0
- net VCC1p2: track 141.2 -> 13.5 mm, vias 25 -> 0
- net (no net): track 103.6 -> 0.00 mm, vias 144 -> 0
- net F_CLK2: track 103.4 -> 0.00 mm
- net F_CLK3: track 103.3 -> 0.00 mm
- net GND: track 89.1 -> 0.00 mm, vias 35 -> 0
- net Net-(P1-Pad5): track 87.4 -> 0.00 mm
- net Net-(P1-Pad3): track 84.8 -> 0.00 mm
- net Net-(P1-Pad1): track 80.2 -> 0.00 mm
- net VCC: track 75.6 -> 0.00 mm
- net Net-(P1-Pad2): track 65.6 -> 0.00 mm, vias 2 -> 0
- net Net-(P1-Pad6): track 64.2 -> 0.00 mm, vias 2 -> 0
- net Net-(P1-Pad4): track 62.6 -> 0.00 mm, vias 2 -> 0
- net /FPGA Configuration Circuitry/JTAG_TDO: track 61.6 -> 0.00 mm
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- removed copper zone on F.Cu, net GND
